Commit message: MoveIt initial setup and configs fixes

File: ros2_rm_robot/dual_rm_gazebo/config/dual_rm_75b_gazebo.urdf.xacro (robot description, xacro)
@@ -1,4 +1,4 @@
 <?xml version="1.0"?>
-<robot xmlns:xacro="http://www.ros.org/wiki/xacro" name="dual_rm_75b_gazebo">
+<robot xmlns:xacro="http://www.ros.org/wiki/xacro" name="dual_rm_75b_description">
     <xacro:include filename="$(find dual_rm_75b_description)/urdf/dual_rm_75b_description.urdf.xacro" />
     <!-- <xacro:include filename="$(find dual_rm_gazebo)/config/dg4f_gazebo_classic.urdf.xacro"/> -->

File: ros2_rm_robot/dual_rm_moveit_config/dual_rm_75b_moveit_config/config/dual_rm_75b_description.ros2_control.xacro (robot description, xacro)
@@ -57,4 +57,11 @@
                 <state_interface name="velocity"/>
             </joint> -->
+            <joint name="l_4c2_gripper_joint">
+                <command_interface name="position"/>
+                <state_interface name="position">
+                  <param name="initial_value">${initial_positions['l_4c2_gripper_joint']}</param>
+                </state_interface>
+                <state_interface name="velocity"/>
+            </joint>
             <joint name="r_joint1">
                 <command_interface name="position"/>
@@ -106,4 +113,11 @@
                 <state_interface name="velocity"/>
             </joint> -->
+            <joint name="r_4c2_gripper_joint">
+                <command_interface name="position"/>
+                <state_interface name="position">
+                  <param name="initial_value">${initial_positions['r_4c2_gripper_joint']}</param>
+                </state_interface>
+                <state_interface name="velocity"/>
+            </joint>
             <joint name="platform_joint">
                 <command_interface name="position"/>
